File: pcb/myCompactKeyboard.kicad_pcb (KiCad board)
At the start: 2 copper layers, 290 parts, among them J1 OLED_128x64, SW1 RotaryEncoder_Switch, SW2 RotaryEncoder_Switch, U1 Raspberry_Pi_Pico

Commit message: placed diodes on pcb
Parts:
- moved D78 339.0 mm to (17.6, -11.9)
- moved D50 320.9 mm to (17.6, 14.3)
- moved D51 309.4 mm to (17.6, 33.3)
- moved D13 287.3 mm to (36.7, 14.3)
- moved D14 280.0 mm to (54.8, 14.3)
- moved D15 272.8 mm to (74.8, 14.3)
- moved D52 267.7 mm to (17.6, 52.4)
- moved D16 267.3 mm to (93.8, 14.3)
- moved D2 265.8 mm to (55.7, -11.9)
- moved D25 265.7 mm to (36.7, 33.3)
- moved D56 265.0 mm to (17.6, 71.4)
- moved D49 263.8 mm to (36.7, 71.4)
- moved D82 263.4 mm to (279.6, -11.9)
- moved D17 263.2 mm to (112.9, 14.3)
- moved D60 262.4 mm to (17.6, 90.5)
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
Commit message: placed all elements on pcb and started wiring
Parts:
- D100, D101, D102, D103, D104, D105, D106, D107, D108, D109, D110, D111, D112, D113, D114, D115, D116, D117, D118, D119, D120, D121, D122, D123, D124, D125, D126, D127, D128, D129, D130, D131, D132, D133, D134, D135, D136, D137, D138, D139, D140, D141, D142, D143, D144, D145, D146, D147, D148, D149, D150, D151, D152, D153, D154, D155, D156, D157, D158, D159, D160, D161, D162, D163, D164, D165, D166, D167, D168, D169, D170, D171, D172, D173, D174, D175, D176, D177, D178, D179, D180, D181, D182, D183, D184, D185, D186, D187, D188, D189, D190, D191, D192, D97, D98, D99: footprint ScottoKeebs_Components:LED_WS2812B -> leds:SK6812MINI-E
- moved D192 238.0 mm to (38.4, 208.9)
- moved U1 230.2 mm to (346.2, 116.2)
- moved D188 228.7 mm to (57.5, 208.9)
- moved D166 214.1 mm to (38.4, 170.8)
- moved D170 213.3 mm to (38.4, 189.9)
- moved D162 200.3 mm to (57.5, 170.8)
- moved D139 196.1 mm to (38.4, 151.8)
- moved D137 195.8 mm to (38.4, 132.7)
- moved D174 193.7 mm to (57.5, 189.9)
- moved D178 189.8 mm to (76.5, 189.9)
- moved D184 185.4 mm to (76.5, 208.9)
- moved D135 180.7 mm to (57.5, 132.7)
- moved J1 179.8 mm to (360.6, 166.5), turned to -90 degrees
- moved D141 176.7 mm to (57.5, 151.8)
- moved D180 173.4 mm to (95.6, 208.9)
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Routing:
- net Col 6: track 0.00 -> 95.4 mm
- net Col 2: track 0.00 -> 94.8 mm
- net Col 3: track 0.00 -> 94.5 mm
- net Col 10: track 0.00 -> 94.4 mm
- net Col 7: track 0.00 -> 94.3 mm
- net Col 11: track 0.00 -> 94.2 mm
- net Col 5: track 0.00 -> 94.2 mm
- net Col 4: track 0.00 -> 94.1 mm
- net Col 8: track 0.00 -> 94.1 mm
- net Col 9: track 0.00 -> 94.0 mm
- net Col 1: track 0.00 -> 34.1 mm
Other:
- board outline added: 3.4 x 3 mm

Commit message: fixed all components placement
Parts:
- moved U1 114.6 mm to (333.4, 2.38)
- moved D82 110.6 mm to (283.8, -21.4), turned to 180 degrees
- moved D1 110.4 mm to (36.7, -19.1)
- moved D10 110.4 mm to (208.1, -19.1)
- moved D100 110.4 mm to (78.6, -9.53)
- moved D101 110.4 mm to (97.6, -9.53)
- moved D102 110.4 mm to (116.7, -9.53)
- moved D103 110.4 mm to (135.7, -9.53)
- moved D104 110.4 mm to (154.8, -9.53)
- moved D105 110.4 mm to (173.8, -9.53)
- moved D106 110.4 mm to (192.9, -9.53)
- moved D107 110.4 mm to (211.9, -9.53)
- moved D108 110.4 mm to (231.0, -9.53)
- moved D11 110.4 mm to (227.2, -19.1)
- moved D2 110.4 mm to (55.7, -19.1)
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Routing:
- net Col 6: track 95.4 -> 0.00 mm
- net Col 2: track 94.8 -> 0.00 mm
- net Col 3: track 94.5 -> 0.00 mm
- net Col 10: track 94.4 -> 0.00 mm
- net Col 7: track 94.3 -> 0.00 mm
- net Col 11: track 94.2 -> 0.00 mm
- net Col 5: track 94.2 -> 0.00 mm
- net Col 4: track 94.1 -> 0.00 mm
- net Col 8: track 94.1 -> 0.00 mm
- net Col 9: track 94.0 -> 0.00 mm
- net Col 1: track 34.1 -> 0.00 mm

Commit message: positioned all Led on the pcb
Parts:
- D100, D101, D102, D103, D104, D105, D106, D107, D108, D109, D110, D111, D112, D113, D114, D115, D116, D117, D118, D119, D120, D121, D122, D123, D124, D125, D126, D127, D128, D129, D130, D131, D132, D133, D134, D135, D136, D137, D138, D139, D140, D141, D142, D143, D144, D145, D146, D147, D148, D149, D150, D151, D152, D153, D154, D155, D156, D157, D158, D159, D160, D161, D162, D163, D164, D165, D166, D167, D168, D169, D170, D171, D172, D173, D174, D175, D176, D177, D178, D179, D180, D181, D182, D183, D184, D185, D186, D187, D188, D189, D190, D191, D192, D97, D98, D99: moved to B.Cu
- moved D122 5.08 mm to (78.6, 47.9), turned to 180 degrees
- moved D124 5.08 mm to (97.6, 47.9), turned to 180 degrees
- moved D126 5.08 mm to (116.7, 47.9), turned to 180 degrees
- moved D128 5.08 mm to (135.7, 47.9), turned to 180 degrees
- moved D130 5.08 mm to (154.8, 47.9), turned to 180 degrees
- moved D132 5.08 mm to (173.8, 47.9), turned to 180 degrees
- moved D134 5.08 mm to (192.9, 47.9), turned to 180 degrees
- moved D136 5.08 mm to (211.9, 47.9), turned to 180 degrees
- moved D138 5.08 mm to (231.0, 47.9), turned to 180 degrees
- moved D139 5.08 mm to (21.4, 47.9), turned to 180 degrees
- moved D140 5.08 mm to (250.0, 47.9), turned to 180 degrees
- moved D141 5.08 mm to (40.5, 47.9), turned to 180 degrees
- moved D143 5.08 mm to (59.5, 47.9), turned to 180 degrees
- moved D144 5.08 mm to (288.1, 47.9), turned to 180 degrees
- moved D145 5.08 mm to (307.2, 47.9), turned to 180 degrees
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Other:
- board size 3.4 x 3 mm -> 359.6 x 138.1 mm

Commit message: flipped all diodes
Parts:
- D1, D10, D11, D12, D13, D14, D15, D16, D17, D18, D19, D2, D20, D21, D22, D23, D24, D25, D26, D27, D28, D29, D3, D30, D31, D32, D33, D34, D35, D36, D37, D38, D39, D4, D40, D41, D42, D43, D44, D45, D46, D47, D48, D49, D5, D50, D51, D52, D53, D54, D55, D56, D57, D58, D59, D6, D60, D61, D62, D63, D64, D65, D66, D67, D68, D69, D7, D70, D71, D72, D73, D74, D75, D76, D77, D78, D79, D8, D80, D81, D82, D83, D84, D85, D86, D87, D88, D89, D9, D90, D91, D92, D93, D94, D95, D96, U1: moved to B.Cu
- moved U1 3.38 mm to (330.0, 2.38), turned to 180 degrees

Commit message: wired all simple keyswitch connections
Parts:
- added J2: AudioJack4, Connector_Audio:Jack_3.5mm_CUI_SJ1-3524N_Horizontal, F.Cu at (270.0, -17.5)
- moved D110 9.53 mm to (288.1, 2.50)
- moved D86 9.53 mm to (312.4, -21.4)
- moved SW1 9.53 mm to (285.6, -2.27)
- moved D111 9.52 mm to (307.2, 2.50)
- moved D82 9.52 mm to (293.4, -21.4)
- moved SW2 9.52 mm to (304.7, -2.27)
Connections:
- U1 pad 1: Row 1 -> R1
- U1 pad 10: Row 8 -> Row 6
- U1 pad 11: Col 1 -> Row 7
- U1 pad 12: Col 2 -> Row 8
- U1 pad 13: unconnected-(U1-GND-Pad13) -> GND
- U1 pad 14: Col 3 -> Col 1
- U1 pad 15: Col 4 -> Col 2
- U1 pad 16: Col 5 -> Col 3
- U1 pad 17: Col 6 -> Col 4
- U1 pad 18: unconnected-(U1-GND-Pad18) -> GND
- U1 pad 19: Col 7 -> Col 5
- U1 pad 2: Row 2 -> R2
- U1 pad 20: Col 8 -> Col 6
- U1 pad 21: Col 9 -> Col 7
- U1 pad 22: Col 10 -> Col 8
- U1 pad 24: Col 11 -> Col 9
- U1 pad 25: Col 12 -> Col 10
- U1 pad 28: unconnected-(U1-GND-Pad28) -> GND
- U1 pad 3: Row 3 -> GND
- U1 pad 31: unconnected-(U1-GPIO26_ADC0-Pad31) -> Col 11
- U1 pad 32: unconnected-(U1-GPIO27_ADC1-Pad32) -> Col 12
- U1 pad 34: unconnected-(U1-GPIO28_ADC2-Pad34) -> T
- U1 pad 38: unconnected-(U1-GND-Pad38) -> GND
- U1 pad 4: Row 3 -> Row 1
- U1 pad 5: Row 4 -> Row 2
- U1 pad 6: Row 5 -> Row 3
- U1 pad 7: Row 6 -> Row 4
- U1 pad 8: unconnected-(U1-GND-Pad8) -> GND
- U1 pad 9: Row 7 -> Row 5
Routing:
- net Net-(D72-A): track 0.00 -> 4.97 mm
- net Net-(D68-A): track 0.00 -> 4.97 mm
- net Net-(D83-A): track 0.00 -> 4.97 mm
- net Net-(D79-A): track 0.00 -> 4.97 mm
- net Net-(D70-A): track 0.00 -> 4.97 mm
- net Net-(D84-A): track 0.00 -> 4.97 mm
- net Net-(D80-A): track 0.00 -> 4.97 mm
- net Net-(D71-A): track 0.00 -> 4.97 mm
- net Net-(D67-A): track 0.00 -> 4.97 mm
- net Net-(D66-A): track 0.00 -> 4.97 mm
- net Net-(D58-A): track 0.00 -> 4.97 mm
- net Net-(D54-A): track 0.00 -> 4.97 mm
- net Net-(D59-A): track 0.00 -> 4.97 mm
- net Net-(D24-A): track 0.00 -> 4.97 mm
- net Net-(D22-A): track 0.00 -> 4.97 mm
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